Commit message: feat: implement ROS 2 autonomous navigation package with SLAM and URDF

File: 01_Robotics_Intelligent_Systems/ROS2_Mobile_Robot_Simulation/src/mobile_robot_nav/urdf/diff_bot.urdf.xacro (robot description, xacro)
@@ -1,60 +1,124 @@
 <?xml version="1.0"?>
 <robot xmlns:xacro="http://www.ros.org/wiki/xacro" name="diff_bot">
+  <!-- Xacro properties -->
+  <xacro:property name="base_length" value="0.3"/>
+  <xacro:property name="base_width" value="0.25"/>
+  <xacro:property name="base_height" value="0.1"/>
+  <xacro:property name="wheel_radius" value="0.05"/>
+  <xacro:property name="wheel_width" value="0.05"/>
+  <xacro:property name="wheel_separation" value="0.25"/>
+  <xacro:property name="lidar_radius" value="0.03"/>
+  <xacro:property name="lidar_height" value="0.06"/>
+  <!-- Base Link -->
   <link name="base_link">
     <visual>
       <geometry>
-        <box size="0.4 0.3 0.1"/>
+        <box size="${base_length} ${base_width} ${base_height}"/>
       </geometry>
       <material name="blue">
-        <color rgba="0 0 1 1"/>
+        <color rgba="0.0 0.0 1.0 1.0"/>
       </material>
+      <origin xyz="0 0 0" rpy="0 0 0"/>
     </visual>
+    <collision>
+      <geometry>
+        <box size="${base_length} ${base_width} ${base_height}"/>
+      </geometry>
+      <origin xyz="0 0 0" rpy="0 0 0"/>
+    </collision>
+    <inertial>
+      <mass value="5.0"/>
+      <inertia ixx="0.1" ixy="0.0" ixz="0.0" iyy="0.1" iyz="0.0" izz="0.1"/>
+      <origin xyz="0 0 0" rpy="0 0 0"/>
+    </inertial>
   </link>
+  <!-- Left Wheel Joint (continuous) -->
+  <joint name="left_wheel_joint" type="continuous">
+    <parent link="base_link"/>
+    <child link="left_wheel"/>
+    <axis xyz="0 1 0"/>
+    <origin xyz="0 ${wheel_separation/2} -${base_height/2 - wheel_radius}" rpy="0 0 0"/>
+  </joint>
+  <!-- Left Wheel Link -->
   <link name="left_wheel">
     <visual>
       <geometry>
-        <cylinder radius="0.1" length="0.05"/>
+        <cylinder radius="${wheel_radius}" length="${wheel_width}"/>
       </geometry>
       <material name="black">
-        <color rgba="0 0 0 1"/>
+        <color rgba="0.0 0.0 0.0 1.0"/>
       </material>
+      <origin xyz="0 0 0" rpy="0 0 0"/>
     </visual>
+    <collision>
+      <geometry>
+        <cylinder radius="${wheel_radius}" length="${wheel_width}"/>
+      </geometry>
+      <origin xyz="0 0 0" rpy="0 0 0"/>
+    </collision>
+    <inertial>
+      <mass value="0.5"/>
+      <inertia ixx="0.01" ixy="0.0" ixz="0.0" iyy="0.01" iyz="0.0" izz="0.01"/>
+      <origin xyz="0 0 0" rpy="0 0 0"/>
+    </inertial>
   </link>
-  <joint name="left_wheel_joint" type="continuous">
+  <!-- Right Wheel Joint (continuous) -->
+  <joint name="right_wheel_joint" type="continuous">
     <parent link="base_link"/>
-    <child link="left_wheel"/>
-    <origin xyz="0 0.175 0" rpy="-1.5708 0 0"/>
-    <axis xyz="0 0 1"/>
+    <child link="right_wheel"/>
+    <axis xyz="0 1 0"/>
+    <origin xyz="0 -${wheel_separation/2} -${base_height/2 - wheel_radius}" rpy="0 0 0"/>
   </joint>
+  <!-- Right Wheel Link -->
   <link name="right_wheel">
     <visual>
       <geometry>
-        <cylinder radius="0.1" length="0.05"/>
+        <cylinder radius="${wheel_radius}" length="${wheel_width}"/>
       </geometry>
       <material name="black">
-        <color rgba="0 0 0 1"/>
+        <color rgba="0.0 0.0 0.0 1.0"/>
       </material>
+      <origin xyz="0 0 0" rpy="0 0 0"/>
     </visual>
+    <collision>
+      <geometry>
+        <cylinder radius="${wheel_radius}" length="${wheel_width}"/>
+      </geometry>
+      <origin xyz="0 0 0" rpy="0 0 0"/>
+    </collision>
+    <inertial>
+      <mass value="0.5"/>
+      <inertia ixx="0.01" ixy="0.0" ixz="0.0" iyy="0.01" iyz="0.0" izz="0.01"/>
+      <origin xyz="0 0 0" rpy="0 0 0"/>
+    </inertial>
   </link>
-  <joint name="right_wheel_joint" type="continuous">
+  <!-- LiDAR Sensor Frame Joint (fixed) -->
+  <joint name="lidar_joint" type="fixed">
     <parent link="base_link"/>
-    <child link="right_wheel"/>
-    <origin xyz="0 -0.175 0" rpy="-1.5708 0 0"/>
-    <axis xyz="0 0 1"/>
+    <child link="laser_frame"/>
+    <origin xyz="${base_length/2} 0 ${base_height/2}" rpy="0 0 0"/>
   </joint>
+  <!-- LiDAR Sensor Frame -->
   <link name="laser_frame">
     <visual>
       <geometry>
-        <cylinder radius="0.05" length="0.04"/>
+        <cylinder radius="${lidar_radius}" length="${lidar_height}"/>
       </geometry>
       <material name="red">
-        <color rgba="1 0 0 1"/>
+        <color rgba="1.0 0.0 0.0 1.0"/>
       </material>
+      <origin xyz="0 0 0" rpy="0 0 0"/>
     </visual>
+    <collision>
+      <geometry>
+        <cylinder radius="${lidar_radius}" length="${lidar_height}"/>
+      </geometry>
+      <origin xyz="0 0 0" rpy="0 0 0"/>
+    </collision>
+    <inertial>
+      <mass value="0.2"/>
+      <inertia ixx="0.001" ixy="0.0" ixz="0.0" iyy="0.001" iyz="0.0" izz="0.001"/>
+      <origin xyz="0 0 0" rpy="0 0 0"/>
+    </inertial>
   </link>
-  <joint name="laser_joint" type="fixed">
-    <parent link="base_link"/>
-    <child link="laser_frame"/>
-    <origin xyz="0.15 0 0.07" rpy="0 0 0"/>
-  </joint>
 </robot>
